File: 00 - Hardware/Power_USB_Batt.sch.kicad_sch (KiCad schematic)
At the start: 36 parts, among them IC1 MAX17048G+T10, J2 USB_C_Receptacle_USB2.0_16P, J4 Header_01x02_2.0mm JST PH, U1 TPS2116DRLR, U2 MIC5219-3.3YM5, U3 USBLC6-2SC6, U4 MCP73831-2-OT

Commit message: updated FDTI cbus connections
Parts:
- removed H1, H2, H3, H4: MountingHole_M3, Project_Footprints:MountingHole_3.2mm_M3_DIN965_Pad, symbol Library:MountingHole_M3
- added H1, H2, H3, H4: MountingHole_Pad_M3, MountingHole:MountingHole_3.2mm_M3_DIN965_Pad_TopBottom, symbol IBA_mechanical_parts:MountingHole_Pad_M3
- added R19, R21: 27, Resistor_SMD:R_0603_1608Metric, symbol Device:R
Connections:
- net GND: now also H1.1, H2.1, H3.1, H4.1
- net USB_D+: now also R19.1; no longer U3.6 (I/O1)
- net USB_D-: now also R21.1; no longer U3.1 (I/O1)
- new net D_N: R21.2, U3.1 (I/O1)
- new net D_P: R19.2, U3.6 (I/O1)
Other:
- note added: "Battery Connection - JST PH 2mm"
- note removed: "Battery Connection - JST"
- moved on the sheet: U3
